Commit message: Add build logs for lexium_cobot_l18s package
- Created stdout_stderr.log to capture installation output and symlink status.
- Added streams.log to log command invocations and their results during the build process.
- Introduced logger_all.log for comprehensive debugging information during the build of the lexium_cobot_l18s package.

File: src/lexium_cobot_l18s/urdf/Lexium_Cobot_L18S002.urdf (robot description, URDF)
Before this commit: robot Lexium_Cobot_L18S002, 7 links, 6 joints
Links:
- link l_Base_Link002: mass None -> 5.0; geometry collision mesh filename=package://lexium_cobot_l18s/meshes/base_link.obj; visual mesh filename=package://lexium_cobot_l18s/meshes/base_link.obj
- link l_Link_012: mass None -> 2.0; geometry collision mesh filename=package://lexium_cobot_l18s/meshes/link_1.obj; visual mesh filename=package://lexium_cobot_l18s/meshes/link_1.obj
- link l_Link_013: mass None -> 2.0; geometry collision mesh filename=package://lexium_cobot_l18s/meshes/link_2.obj; visual mesh filename=package://lexium_cobot_l18s/meshes/link_2.obj
- link l_Link_014: mass None -> 1.5; geometry collision mesh filename=package://lexium_cobot_l18s/meshes/link_3.obj; visual mesh filename=package://lexium_cobot_l18s/meshes/link_3.obj
- link l_Link_015: mass None -> 1.0; geometry collision mesh filename=package://lexium_cobot_l18s/meshes/link_4.obj; visual mesh filename=package://lexium_cobot_l18s/meshes/link_4.obj
- link l_Link_016: mass None -> 0.8; geometry collision mesh filename=package://lexium_cobot_l18s/meshes/link_5.obj; visual mesh filename=package://lexium_cobot_l18s/meshes/link_5.obj
- link l_Link_017: mass None -> 0.5; geometry collision mesh filename=package://lexium_cobot_l18s/meshes/link_6.obj; visual mesh filename=package://lexium_cobot_l18s/meshes/link_6.obj
Joints:
- joint l_Base_Link002__to__l_Link_012: limit effort=0.0 velocity=0.0 -> (none)
- joint l_Link_012__to__l_Link_013: limit effort=0.0 velocity=0.0 -> (none)
- joint l_Link_013__to__l_Link_014: limit effort=0.0 velocity=0.0 -> (none)
- joint l_Link_014__to__l_Link_015: limit effort=0.0 velocity=0.0 -> (none)
- joint l_Link_015__to__l_Link_016: limit effort=0.0 velocity=0.0 -> (none)
- joint l_Link_016__to__l_Link_017: limit effort=0.0 velocity=0.0 -> (none)

Commit message: Add Gazebo launch configuration and ros2_control URDF for Lexium Cobot L18S
- Introduced a new Gazebo launch file for the Lexium Cobot L18S, enabling simulation with ros2_control.
- Created a URDF Xacro file defining the ros2_control hardware interface for the robot, including command and state interfaces for multiple joints.

File: src/lexium_cobot_l18s/urdf/Lexium_Cobot_L18S002.urdf (robot description, URDF)
Before this commit: robot Lexium_Cobot_L18S002, 7 links, 6 joints
Links:
- added link world
- link l_Base_Link002: geometry collision box size=0.19 0.20 0.05; visual mesh filename=package://lexium_cobot_l18s/meshes/base_link.obj
- link l_Link_012: geometry collision box size=0.16 0.16 0.20; visual mesh filename=package://lexium_cobot_l18s/meshes/link_1.obj
- link l_Link_013: geometry collision box size=0.20 0.16 0.65; visual mesh filename=package://lexium_cobot_l18s/meshes/link_2.obj
- link l_Link_014: geometry collision box size=0.13 0.12 0.51; visual mesh filename=package://lexium_cobot_l18s/meshes/link_3.obj
- link l_Link_015: geometry collision box size=0.10 0.10 0.13; visual mesh filename=package://lexium_cobot_l18s/meshes/link_4.obj
- link l_Link_016: geometry collision box size=0.13 0.10 0.10; visual mesh filename=package://lexium_cobot_l18s/meshes/link_5.obj
- link l_Link_017: geometry collision box size=0.05 0.09 0.10; visual mesh filename=package://lexium_cobot_l18s/meshes/link_6.obj
Joints:
- added joint world__to__l_Base_Link002: type fixed, parent world, child l_Base_Link002, origin xyz=0.0 0.0 0.0 rpy=0 0 0
- joint l_Base_Link002__to__l_Link_012: limit (none) -> effort=100.0 velocity=2.0
- joint l_Link_012__to__l_Link_013: limit (none) -> effort=80.0 velocity=2.0
- joint l_Link_013__to__l_Link_014: limit (none) -> effort=60.0 velocity=2.5
- joint l_Link_014__to__l_Link_015: limit (none) -> effort=30.0 velocity=3.0
- joint l_Link_015__to__l_Link_016: limit (none) -> effort=15.0 velocity=3.5
- joint l_Link_016__to__l_Link_017: limit (none) -> effort=10.0 velocity=4.0

File: src/lexium_cobot_l18s/urdf/Lexium_Cobot_L18S002_wrapper.urdf.xacro (robot description, xacro)
@@ -1,5 +1,11 @@
 <?xml version="1.0" encoding="utf-8"?>
 <robot xmlns:xacro="http://www.ros.org/wiki/xacro" name="Lexium_Cobot_L18S002">
+    <xacro:arg name="use_ros2_control" default="false"/>
+    <xacro:arg name="controllers_file" default=""/>
     <xacro:include filename="Lexium_Cobot_L18S002.urdf"/>
     <xacro:include filename="Lexium_Cobot_L18S002_sensors.urdf.xacro"/>
+    <xacro:include filename="Lexium_Cobot_L18S002_ros2_control.urdf.xacro"/>
+    <xacro:if value="$(arg use_ros2_control)">
+      <xacro:lexium_ros2_control controllers_file="$(arg controllers_file)"/>
+    </xacro:if>
 </robot>

Commit message: update link inertial properties and joint limits in cobot URDF

File: src/lexium_cobot_l18s/urdf/Lexium_Cobot_L18S002.urdf (robot description, URDF)
Before this commit: robot Lexium_Cobot_L18S002, 8 links, 7 joints
Links:
- link l_Base_Link002: mass 5.0 -> 7.5
- link l_Link_012: mass 2.0 -> 8.5
- link l_Link_013: mass 2.0 -> 10.5
- link l_Link_014: mass 1.5 -> 4.5
- link l_Link_015: mass 1.0 -> 2.0
- link l_Link_016: mass 0.8 -> 1.2
- link l_Link_017: mass 0.5 -> 0.8
Joints:
- joint l_Base_Link002__to__l_Link_012: limit effort=100.0 velocity=2.0 -> effort=300.0 velocity=2.0944
- joint l_Link_012__to__l_Link_013: limit effort=80.0 velocity=2.0 -> lower=-1.48353 upper=4.62512 effort=300.0 velocity=2.0944; type continuous -> revolute
- joint l_Link_013__to__l_Link_014: limit effort=60.0 velocity=2.5 -> lower=-3.05433 upper=3.05433 effort=150.0 velocity=3.1416; type continuous -> revolute
- joint l_Link_014__to__l_Link_015: limit effort=30.0 velocity=3.0 -> lower=-1.48353 upper=4.62512 effort=80.0 velocity=3.1416; type continuous -> revolute
- joint l_Link_015__to__l_Link_016: limit effort=15.0 velocity=3.5 -> effort=40.0 velocity=3.1416
- joint l_Link_016__to__l_Link_017: limit effort=10.0 velocity=4.0 -> effort=40.0 velocity=3.1416

Commit message: refactor: update robot joint limits, types, and add tool0 frame to URDF, SRDF, and MoveIt configs

File: src/lexium_cobot_l18s/urdf/Lexium_Cobot_L18S002.urdf (robot description, URDF)
Before this commit: robot Lexium_Cobot_L18S002, 8 links, 7 joints
Links:
- added link tool0
Joints:
- added joint l_Link_017__to__tool0: type fixed, parent l_Link_017, child tool0, origin xyz=0.0 0.0 0.039 rpy=0 0 0
- joint l_Base_Link002__to__l_Link_012: limit effort=300.0 velocity=2.0944 -> lower=-4.71239 upper=4.71239 effort=300.0 velocity=2.0944; type continuous -> revolute
- joint l_Link_013__to__l_Link_014: limit lower=-3.05433 upper=3.05433 effort=150.0 velocity=3.1416 -> lower=-3.05433 upper=3.05433 effort=150.0 velocity=2.0944
- joint l_Link_015__to__l_Link_016: limit effort=40.0 velocity=3.1416 -> lower=-4.71239 upper=4.71239 effort=40.0 velocity=3.1416; type continuous -> revolute
- joint l_Link_016__to__l_Link_017: limit effort=40.0 velocity=3.1416 -> lower=-4.71239 upper=4.71239 effort=40.0 velocity=3.1416; type continuous -> revolute
