Commit message: feat: add mock hardware support and launch configuration for ros2_control

File: src/lexium_cobot_l18s/urdf/Lexium_Cobot_L18S002_ros2_control.urdf.xacro (robot description, xacro)
@@ -1,13 +1,21 @@
 <?xml version="1.0"?>
 <robot xmlns:xacro="http://www.ros.org/wiki/xacro">
-  <!-- ros2_control hardware for Gazebo Sim (gz_ros2_control). Included only when use_ros2_control=true -->
-  <xacro:macro name="lexium_ros2_control" params="controllers_file use_sim:=true">
+  <!-- ros2_control configuration for Mock Hardware and Gazebo Sim (gz_ros2_control) -->
+  <xacro:macro name="lexium_ros2_control" params="controllers_file:='' use_sim:=true use_mock_hardware:=false initial_positions:=${dict()}">
     <ros2_control name="LexiumCobotSystem" type="system">
       <hardware>
-        <plugin>gz_ros2_control/GazeboSimSystem</plugin>
+        <xacro:if value="${use_mock_hardware}">
+          <plugin>mock_components/GenericSystem</plugin>
+          <param name="calculate_dynamics">true</param>
+        </xacro:if>
+        <xacro:unless value="${use_mock_hardware}">
+          <plugin>gz_ros2_control/GazeboSimSystem</plugin>
+        </xacro:unless>
       </hardware>
       <joint name="l_Base_Link002__to__l_Link_012">
         <command_interface name="position"/>
-        <state_interface name="position"/>
+        <state_interface name="position">
+          <param name="initial_value">${initial_positions.get('l_Base_Link002__to__l_Link_012', 0.0)}</param>
+        </state_interface>
         <state_interface name="velocity"/>
         <state_interface name="effort"/>
@@ -15,5 +23,7 @@
       <joint name="l_Link_012__to__l_Link_013">
         <command_interface name="position"/>
-        <state_interface name="position"/>
+        <state_interface name="position">
+          <param name="initial_value">${initial_positions.get('l_Link_012__to__l_Link_013', 0.0)}</param>
+        </state_interface>
         <state_interface name="velocity"/>
         <state_interface name="effort"/>
@@ -21,5 +31,7 @@
       <joint name="l_Link_013__to__l_Link_014">
         <command_interface name="position"/>
-        <state_interface name="position"/>
+        <state_interface name="position">
+          <param name="initial_value">${initial_positions.get('l_Link_013__to__l_Link_014', 0.0)}</param>
+        </state_interface>
         <state_interface name="velocity"/>
         <state_interface name="effort"/>
@@ -27,5 +39,7 @@
       <joint name="l_Link_014__to__l_Link_015">
         <command_interface name="position"/>
-        <state_interface name="position"/>
+        <state_interface name="position">
+          <param name="initial_value">${initial_positions.get('l_Link_014__to__l_Link_015', 0.0)}</param>
+        </state_interface>
         <state_interface name="velocity"/>
         <state_interface name="effort"/>
@@ -33,5 +47,7 @@
       <joint name="l_Link_015__to__l_Link_016">
         <command_interface name="position"/>
-        <state_interface name="position"/>
+        <state_interface name="position">
+          <param name="initial_value">${initial_positions.get('l_Link_015__to__l_Link_016', 0.0)}</param>
+        </state_interface>
         <state_interface name="velocity"/>
         <state_interface name="effort"/>
@@ -39,14 +55,18 @@
       <joint name="l_Link_016__to__l_Link_017">
         <command_interface name="position"/>
-        <state_interface name="position"/>
+        <state_interface name="position">
+          <param name="initial_value">${initial_positions.get('l_Link_016__to__l_Link_017', 0.0)}</param>
+        </state_interface>
         <state_interface name="velocity"/>
         <state_interface name="effort"/>
       </joint>
     </ros2_control>
-    <gazebo>
-      <plugin filename="libgz_ros2_control-system.so" name="gz_ros2_control::GazeboSimROS2ControlPlugin">
-        <parameters>${controllers_file}</parameters>
-      </plugin>
-    </gazebo>
+    <xacro:if value="${use_sim and not use_mock_hardware}">
+      <gazebo>
+        <plugin filename="libgz_ros2_control-system.so" name="gz_ros2_control::GazeboSimROS2ControlPlugin">
+          <parameters>${controllers_file}</parameters>
+        </plugin>
+      </gazebo>
+    </xacro:if>
   </xacro:macro>
 </robot>

File: src/lexium_cobot_l18s/urdf/Lexium_Cobot_L18S002_wrapper.urdf.xacro (robot description, xacro)
@@ -2,4 +2,6 @@
 <robot xmlns:xacro="http://www.ros.org/wiki/xacro" name="Lexium_Cobot_L18S002">
     <xacro:arg name="use_ros2_control" default="false"/>
+    <xacro:arg name="use_mock_hardware" default="false"/>
+    <xacro:arg name="use_sim" default="true"/>
     <xacro:arg name="controllers_file" default=""/>
     <xacro:include filename="Lexium_Cobot_L18S002.urdf"/>
@@ -7,5 +9,5 @@
     <xacro:include filename="Lexium_Cobot_L18S002_ros2_control.urdf.xacro"/>
     <xacro:if value="$(arg use_ros2_control)">
-      <xacro:lexium_ros2_control controllers_file="$(arg controllers_file)"/>
+      <xacro:lexium_ros2_control controllers_file="$(arg controllers_file)" use_sim="$(arg use_sim)" use_mock_hardware="$(arg use_mock_hardware)"/>
     </xacro:if>
 </robot>

Commit message: feat: add support for modular gripper and vacuum end-effector tools

File: src/lexium_cobot_l18s/urdf/Lexium_Cobot_L18S002_ros2_control.urdf.xacro (robot description, xacro)
@@ -2,5 +2,5 @@
 <robot xmlns:xacro="http://www.ros.org/wiki/xacro">
   <!-- ros2_control configuration for Mock Hardware and Gazebo Sim (gz_ros2_control) -->
-  <xacro:macro name="lexium_ros2_control" params="controllers_file:='' use_sim:=true use_mock_hardware:=false initial_positions:=${dict()}">
+  <xacro:macro name="lexium_ros2_control" params="controllers_file:='' use_sim:=true use_mock_hardware:=false tool_type:=none initial_positions:=${dict()}">
     <ros2_control name="LexiumCobotSystem" type="system">
       <hardware>
@@ -60,4 +60,21 @@
         <state_interface name="effort"/>
       </joint>
+      <!-- Gripper Joints (if attached) -->
+      <xacro:if value="${tool_type == 'gripper' or tool_type == 'parallel_gripper'}">
+        <joint name="gripper_finger_left_joint">
+          <command_interface name="position"/>
+          <state_interface name="position">
+            <param name="initial_value">0.0</param>
+          </state_interface>
+          <state_interface name="velocity"/>
+          <state_interface name="effort"/>
+        </joint>
+        <joint name="gripper_finger_right_joint">
+          <param name="mimic">gripper_finger_left_joint</param>
+          <param name="multiplier">1.0</param>
+          <state_interface name="position"/>
+          <state_interface name="velocity"/>
+        </joint>
+      </xacro:if>
     </ros2_control>
     <xacro:if value="${use_sim and not use_mock_hardware}">

File: src/lexium_cobot_l18s/urdf/Lexium_Cobot_L18S002_wrapper.urdf.xacro (robot description, xacro)
@@ -5,9 +5,15 @@
     <xacro:arg name="use_sim" default="true"/>
     <xacro:arg name="controllers_file" default=""/>
+    <xacro:arg name="tool_type" default="none"/>
+    <!-- Base Robot Description -->
     <xacro:include filename="Lexium_Cobot_L18S002.urdf"/>
     <xacro:include filename="Lexium_Cobot_L18S002_sensors.urdf.xacro"/>
+    <!-- End-Effector / Tool Framework -->
+    <xacro:include filename="Lexium_Cobot_L18S002_tools.urdf.xacro"/>
+    <xacro:lexium_tool_attachment tool_type="$(arg tool_type)" parent="tool0"/>
+    <!-- ros2_control Hardware Interface -->
     <xacro:include filename="Lexium_Cobot_L18S002_ros2_control.urdf.xacro"/>
     <xacro:if value="$(arg use_ros2_control)">
-      <xacro:lexium_ros2_control controllers_file="$(arg controllers_file)" use_sim="$(arg use_sim)" use_mock_hardware="$(arg use_mock_hardware)"/>
+      <xacro:lexium_ros2_control controllers_file="$(arg controllers_file)" use_sim="$(arg use_sim)" use_mock_hardware="$(arg use_mock_hardware)" tool_type="$(arg tool_type)"/>
     </xacro:if>
 </robot>

Commit message: feat: add pick-and-place workcell demonstration package and test scripts for Lexium cobot

File: src/lexium_cobot_l18s/urdf/Lexium_Cobot_L18S002_ros2_control.urdf.xacro (robot description, xacro)
@@ -63,5 +63,8 @@
       <xacro:if value="${tool_type == 'gripper' or tool_type == 'parallel_gripper'}">
         <joint name="gripper_finger_left_joint">
-          <command_interface name="position"/>
+          <command_interface name="position">
+            <!-- High proportional gain so GazeboSimSystem aggressively tracks position setpoints -->
+            <param name="position_proportional_gain">10000.0</param>
+          </command_interface>
           <state_interface name="position">
             <param name="initial_value">0.0</param>
@@ -70,4 +73,5 @@
           <state_interface name="effort"/>
         </joint>
+        <!-- Right finger mimics left finger — MUST NOT have command_interface (ros2_control aborts) -->
         <joint name="gripper_finger_right_joint">
           <param name="mimic">gripper_finger_left_joint</param>
@@ -75,4 +79,5 @@
           <state_interface name="position"/>
           <state_interface name="velocity"/>
+          <state_interface name="effort"/>
         </joint>
       </xacro:if>

File: src/lexium_cobot_l18s/urdf/tools/generic_parallel_gripper.urdf.xacro (robot description, xacro)
@@ -44,7 +44,7 @@
       <!-- Collision geometry -->
       <collision>
-        <origin xyz="0.0 0.0 0.036" rpy="0 0 0"/>
+        <origin xyz="0.0 0.0 0.032" rpy="0 0 0"/>
         <geometry>
-          <box size="0.080 0.115 0.072"/>
+          <box size="0.075 0.095 0.064"/>
         </geometry>
       </collision>
@@ -103,6 +103,7 @@
       <origin xyz="0.0 0.020 0.068" rpy="0 0 0"/>
       <axis xyz="0 1 0"/>
-      <limit lower="0.0" upper="0.040" effort="100.0" velocity="0.15"/>
-      <dynamics damping="1.0" friction="0.2"/>
+      <limit lower="-0.010" upper="0.040" effort="100.0" velocity="0.15"/>
+      <!-- Low damping/friction so GazeboSimSystem position controller can drive the joint freely -->
+      <dynamics damping="0.1" friction="0.01"/>
     </joint>
     <!-- Right Finger -->
@@ -150,7 +151,8 @@
       <origin xyz="0.0 -0.020 0.068" rpy="0 0 0"/>
       <axis xyz="0 -1 0"/>
-      <limit lower="0.0" upper="0.040" effort="100.0" velocity="0.15"/>
+      <limit lower="-0.010" upper="0.040" effort="100.0" velocity="0.15"/>
       <mimic joint="${prefix}finger_left_joint" multiplier="1.0" offset="0.0"/>
-      <dynamics damping="1.0" friction="0.2"/>
+      <!-- Low damping/friction so GazeboSimSystem position controller can drive the joint freely -->
+      <dynamics damping="0.1" friction="0.01"/>
     </joint>
     <!-- Tool Center Point (TCP) / Grasp Center Frame -->
@@ -164,4 +166,5 @@
     <gazebo reference="${prefix}base_link">
       <material>Gazebo/DarkGrey</material>
+      <self_collide>false</self_collide>
     </gazebo>
     <gazebo reference="${prefix}finger_left">
@@ -169,6 +172,7 @@
       <kp>1000000.0</kp>
       <kd>1.0</kd>
-      <mu1>1.5</mu1>
-      <mu2>1.5</mu2>
+      <mu1>10.0</mu1>
+      <mu2>10.0</mu2>
+      <self_collide>false</self_collide>
     </gazebo>
     <gazebo reference="${prefix}finger_right">
@@ -176,6 +180,7 @@
       <kp>1000000.0</kp>
       <kd>1.0</kd>
-      <mu1>1.5</mu1>
-      <mu2>1.5</mu2>
+      <mu1>10.0</mu1>
+      <mu2>10.0</mu2>
+      <self_collide>false</self_collide>
     </gazebo>
   </xacro:macro>
